File: schematics/circuit schematics/circuit schematics.sch (KiCad schematic (older format))
At the start: 24 parts

Commit message: IR sensor and started motor circuit
Parts:
- removed BT4: RMotor, symbol Device:Battery
- added 3v3: D_Zener, symbol Device:D_Zener
- added C1: 2.3n, symbol pspice:C
- added C2: 230p, symbol pspice:C
- added C3: 470n, symbol pspice:C
- added D? (x2): DIODE, symbol pspice:DIODE
- added Q?: Q_Photo_NPN, symbol Device:Q_Photo_NPN
- added R1, R2, R4: 100k, symbol Device:R
- added R3, R5, R? (x4): 1k, symbol Device:R
- added R6, R7, R8: 33k, symbol Device:R
- added R? (x4): 330, symbol Device:R
- added U1, U2, U3, U4: TL082, symbol Amplifier_Operational:TL082
- added U?: LT1161, symbol LT1161:LT1161
- added U? (x2): MCT6, symbol mct6_custom:MCT6
- BT3: value LMotor -> Motors
- D?: symbol TSHA5203:TSHA5203 -> circuit-schematics-rescue:TSHA5203-TSHA5203
- U?: symbol TCRT5000:TCRT5000 -> circuit-schematics-rescue:TCRT5000-TCRT5000
- renumbered BT5 to BT4
Connections:
- net labels added: +3.3V, BP_Pin, BP_outLB, BP_outLF, BP_outRB, BP_outRF
- net labels removed: BAT_5, GNDA
- wire segments 78 -> 169
Other:
- note added: "IR Detector"
- moved on the sheet: BT1, BT2, BT3, BT4, R?, RV?, U?
