File: schematics/circuit schematics/circuit schematics.sch (KiCad schematic (older format))
At the start: 97 parts, among them J1 USB Programmer, M1 Motor_DC, M2 Motor_DC, M3 Large Servo, M4 Small Servo, Q1 VN2222LL, Q2 Q_Photo_NPN, Q3 VN2222LL, Q4 Q_Photo_NPN, Q5 VN2222LL, Q6 VN2222LL, U1 TL082, U10 LM7833_TO220, U11 IRFZ44, U12 IRFZ44, U13 HC-SR04, U14 TCRT5000, U15 IRFZ44, U16 IRFZ44, U17 TL082, U18 LM311, U19 IRFZ44, U2 TL082, U20 IRFZ44, U21 TL082, U22 L7805, U23 TL082, U24 LM311, U25 TL082, U3 TL082, U4 TL082, U5 LM7805_TO220, U6 MCT6, U7 MCT6, U8 IRFZ44, U9 IRFZ44

Commit message: added text labels to small circuits
Parts:
- BP1: symbol Custom~Parts:STM32_BluePill -> circuit-schematics-rescue:STM32_BluePill-Custom~Parts
- D3: symbol circuit-schematics-rescue:TSHA5203-TSHA5203 -> circuit-schematics-rescue:TSHA5203-TSHA5203-circuit-schematics-rescue
- J?: symbol bp_display:BP_Display -> circuit-schematics-rescue:BP_Display-bp_display
- LT1: symbol LT1161_all-pins:LT1161 -> circuit-schematics-rescue:LT1161-LT1161_all-pins
- U11, U12, U15, U16, U19, U20, U8, U9: symbol IRFZ44:IRFZ44 -> circuit-schematics-rescue:IRFZ44-IRFZ44
- U13: symbol HC-SR04:HC-SR04 -> circuit-schematics-rescue:HC-SR04-HC-SR04
- U14: symbol circuit-schematics-rescue:TCRT5000-TCRT5000 -> circuit-schematics-rescue:TCRT5000-TCRT5000-circuit-schematics-rescue
Other:
- note added: "Arm Servos"
- note added: "Control Switch\n"
- note added: "Display\n"
- note added: "Sonar Sensor"
Changed lines of the file:
@@
 	6850 4450 6850 4700
 $Comp
-L circuit-schematics-rescue:TCRT5000-TCRT5000 U14
+L circuit-schematics-rescue:TCRT5000-TCRT5000-circuit-schematics-rescue U14
 U 1 1 5EE92FBF
 P 7250 4800
@@
 	12300 4200 12300 4100
 $Comp
-L circuit-schematics-rescue:TSHA5203-TSHA5203 D3
+L circuit-schematics-rescue:TSHA5203-TSHA5203-circuit-schematics-rescue D3
 U 1 1 5EEEF279
 P 12300 4500
@@
 Optoisolators and Gate Driver
 $Comp
-L IRFZ44:IRFZ44 U8
+L circuit-schematics-rescue:IRFZ44-IRFZ44 U8
 U 1 1 5EEE04A7
 P 3300 9000
@@
 $EndComp
 $Comp
-L IRFZ44:IRFZ44 U11
+L circuit-schematics-rescue:IRFZ44-IRFZ44 U11
 U 1 1 5EEE61B9
 P 4300 9000
@@
 $EndComp
 $Comp
-L IRFZ44:IRFZ44 U9
+L circuit-schematics-rescue:IRFZ44-IRFZ44 U9
 U 1 1 5EEEA055
 P 3300 10200
@@
 $EndComp
 $Comp
-L IRFZ44:IRFZ44 U12
+L circuit-schematics-rescue:IRFZ44-IRFZ44 U12
 U 1 1 5EEEA94B
 P 4300 10200
@@
 	5450 9300 5450 8800
 $Comp
-L IRFZ44:IRFZ44 U16
+L circuit-schematics-rescue:IRFZ44-IRFZ44 U16
 U 1 1 5F2BA848
 P 7950 10250
@@
 $EndComp
 $Comp
-L IRFZ44:IRFZ44 U15
+L circuit-schematics-rescue:IRFZ44-IRFZ44 U15
 U 1 1 5F2C7B96
 P 7950 9000
@@
 $EndComp
 $Comp
-L IRFZ44:IRFZ44 U19
+L circuit-schematics-rescue:IRFZ44-IRFZ44 U19
 U 1 1 5F2E0E0B
 P 9350 9000
@@
 $EndComp
 $Comp
-L IRFZ44:IRFZ44 U20
+L circuit-schematics-rescue:IRFZ44-IRFZ44 U20
 U 1 1 5F2E1AAB
 P 9350 10250
@@
 BAT_3
 $Comp
-L LT1161_all-pins:LT1161 LT1
+L circuit-schematics-rescue:LT1161-LT1161_all-pins LT1
 U 1 1 5F6EDE90
 P 4400 4550
@@
 $EndComp
 $Comp
-L Custom~Parts:STM32_BluePill BP1
+L circuit-schematics-rescue:STM32_BluePill-Custom~Parts BP1
 U 1 1 609C409C
 P 14550 2650
@@
 	13050 2050 13650 2050
 $Comp
-L HC-SR04:HC-SR04 U13
+L circuit-schematics-rescue:HC-SR04-HC-SR04 U13
 U 1 1 60CD3600
 P 7200 1800
@@
 BP_out_Sonar
 $Comp
-L bp_display:BP_Display J?
+L circuit-schematics-rescue:BP_Display-bp_display J?
 U 1 1 617ECB45
 P 11000 2250
@@
 Text Label 11200 2200 0    50   ~ 0
 GND_Disp
+Text Notes 6800 1050 0    50   ~ 0
+Sonar Sensor
+Text Notes 8950 1000 0    50   ~ 0
+Arm Servos
+Text Notes 11600 1100 0    50   ~ 0
+Control Switch\n
+Text Notes 11600 1500 0    50   ~ 0
+Control Switch\n
+Text Notes 11650 2400 0    50   ~ 0
+Display\n
 $EndSCHEMATC

Commit message: added text labels to circuits maybe
Parts:
- BP1: symbol circuit-schematics-rescue:STM32_BluePill-Custom~Parts -> Custom_Parts:STM32_BluePill
- U6, U7: symbol circuit-schematics-rescue:MCT6-mct6_custom -> circuit-schematics-rescue:MCT6-mct6_custom-circuit-schematics-rescue
Changed lines of the file:
@@
 	1550 4750 2100 4750
 $Comp
-L circuit-schematics-rescue:MCT6-mct6_custom U7
+L circuit-schematics-rescue:MCT6-mct6_custom-circuit-schematics-rescue U7
 U 1 1 5F88C55B
 P 2350 4950
@@
 	2750 4400 2950 4400
 $Comp
-L circuit-schematics-rescue:MCT6-mct6_custom U6
+L circuit-schematics-rescue:MCT6-mct6_custom-circuit-schematics-rescue U6
 U 1 1 5FFC5DD3
 P 2350 4200
@@
 $EndComp
 $Comp
-L circuit-schematics-rescue:STM32_BluePill-Custom~Parts BP1
+L Custom_Parts:STM32_BluePill BP1
 U 1 1 609C409C
 P 14550 2650
