File: schematics/circuit schematics/circuit schematicsv1.2.sch (KiCad schematic (older format))
At the start: 116 parts, among them J1 USB Programmer, M1 Motor_DC, M2 Motor_DC, M3 Large Servo, M4 Small Servo, Q1 VN2222LL, Q2 Q_Photo_NPN, Q3 VN2222LL, Q4 Q_Photo_NPN, Q5 VN2222LL, Q6 VN2222LL, U1 TL082, U10 LM7833_TO220, U11 IRFZ44, U12 IRFZ44, U13 HC-SR04, U14 TCRT5000, U15 IRFZ44, U16 IRFZ44, U17 TL082, U18 LM311, U19 IRFZ44, U2 TL082, U20 IRFZ44, U21 TL082, U24 LM311, U3 TL082, U4 TL082, U5 LM7805_TO220, U6 MCT6, U7 MCT6, U8 IRFZ44, U9 IRFZ44

Commit message: added v1.2
Connections:
- net labels added: BP_in_limit
- wire segments 436 -> 437
Other:
- note added: "Sonar Sensor"
Changed lines of the file:
@@
 Text Label 13050 5700 2    50   ~ 0
 BP_outLS
-Text Label 14800 6300 0    50   ~ 0
-BP_outSS
 Text Label 10700 4200 0    50   ~ 0
 BP_IR1
@@
 Wire Wire Line
 	7100 2100 7100 2500
+Text Notes 12900 3350 0    50   ~ 0
+Sonar Sensor
+Text Label 14800 6300 0    50   ~ 0
+BP_outSS
+Wire Wire Line
+	13050 6750 12400 6750
+Text Label 12400 6750 2    50   ~ 0
+BP_in_limit
 $EndSCHEMATC

Commit message: a lot of stuff lol
Parts:
- removed R?: 33k, symbol Device:R
- removed R?: 47k, symbol Device:R
- added BT5: Motors (9 V), symbol Device:Battery
- added C? (x2): 2.3n, symbol pspice:C
- added C? (x2): 470 nf, symbol Device:CP
- added D?: TSHA5203, LEDRD254W55D595H1320, symbol circuit-schematicsv1.2-rescue:TSHA5203-TSHA5203-circuit-schematics-rescue-circu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
- added R?: 47k, symbol Device:R
- added R?: 100, symbol Device:R
- added R? (x2): R, symbol Device:R
- added U?: TCRT5000, OPTO_TCRT5000, symbol TCRT5000:TCRT5000
- added U?: LM7805_TO220, Package_TO_SOT_THT:TO-220-3_Vertical, symbol Regulator_Linear:LM7805_TO220
- added U?: LM7833_TO220, Package_TO_SOT_THT:TO-220-3_Vertical, symbol Regulator_Linear:LM7805_TO220
- BT3: value Motors (18 V) -> Motors (9 V)
- R23, R?: value 100k -> R
- R?: value 100 -> R
Connections:
- net labels added: GNDREF
- wire segments 437 -> 470
Other:
- note added: "5V"
- note added: "9V"
- note added: "There is a better circuit for this part"
- note added: "Values to be determined"
- note removed: "5.2875 V"
- moved on the sheet: 3v1, 3v?, BT1, BT2, BT3, BT4, C4, D3, Q4, Q?, R17, R18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
